File: ursus-arctos/ursus-arctos.kicad_sch (KiCad schematic)
At the start: 61 parts, among them J1 Conn_01x02, J2 Conn_01x30_Female, J3 Conn_01x08, SW1 RESET, SW19 EVQWGD0001, U1 Seeeduino XIAO BLE

Commit message: cleanup ursus arctos design
Parts:
- removed C1, C10, C11, C12, C14, C15, C16, C3, C5, C6, C7, C8, C9: 1uF, Capacitor_SMD:C_0805_2012Metric, symbol Device:C_Small
- removed C13: 16.1uF, Capacitor_SMD:C_0805_2012Metric, symbol Device:C_Small
- removed C17: 4.7uF, Capacitor_SMD:C_0805_2012Metric, symbol Device:C_Small
- removed C2, C4: 2.2uF, Capacitor_SMD:C_0805_2012Metric, symbol Device:C_Small
- removed DS1: D, Diode_SMD:D_0805_2012Metric, symbol Device:D_Schottky_Small
- removed J2: Conn_01x30_Female, Connector_FFC-FPC:Hirose_FH12-30S-0.5SH_1x30-1MP_P0.50mm_Horizontal, symbol Connector:Conn_01x30_Female
- removed J3: Conn_01x08, Connector_PinHeader_2.54mm:PinHeader_1x08_P2.54mm_Vertical, symbol Connector_Generic:Conn_01x08
- removed SW1: RESET, Jumper:SolderJumper-2_P1.3mm_Open_TrianglePad1.0x1.5mm, symbol Switch:SW_Push
- added D? (x18): 1N4148W, Diode_SMD:D_0805_2012Metric, symbol Device:D_Small_Filled
- added J?: Conn_01x02, Connector_JST:JST_PH_S2B-PH-K_1x02_P2.00mm_Horizontal, symbol Connector_Generic:Conn_01x02
- added JP?: RE_SJ, Jumper:SolderJumper-3_P2.0mm_Open_TrianglePad1.0x1.5mm, symbol Jumper:SolderJumper_3_Open
- added S? (x18): SW_SPST, switches:Choc_PG1350_Choc_Spacing, symbol Switch:SW_SPST
- added SW?: EVQWGD0001, Encoder:RollerEncoder_Panasonic_EVQWGD001, symbol Device:RotaryEncoder_Switch
- added U?: Seeeduino XIAO BLE, reee:xiao-ble, symbol reee:xiao-ble
- JP1: value SolderJumper_3_Open -> (none)
- renumbered SW19 to SW1
Connections:
- net GND: now also JP?.1 (A); no longer U1.13 (GND), U1.20 (GND)
- net at D16.2 (A), S16.2 (B): now also SW1.S1; no longer SW1.S2
- net L_RE-C: now reaches JP1.2 (C), SW1.C
- net L_RE-C: now also SW?.C
- net +3V3 renamed L_3V3
- net BAT+ renamed L_BAT+
- net BAT- renamed L_BAT-
- net C0 renamed L_C0
- net C1 renamed L_C1
- net C2 renamed L_C2
- net L_C2: now also SW1.S2; no longer SW1.S1
- net C3 renamed L_C3
- net C4 renamed L_C4
- net R0 renamed L_R0
- net R1 renamed L_R1
- net R2 renamed L_R2
- net R3 renamed L_R3
- net RE_A renamed L_RE-A
- net L_RE-A: now also SW?.A
- net RE_B renamed L_RE-B
- net L_RE-B: now also SW?.B
- new net: D?.2 (A), S?.2 (B) (x17)
- new net: D?.2 (A), S?.2 (B), SW?.S1
- new net L_GND: U1.13 (GND)
- new net R_3V3: JP?.3 (B), U?.12 (3V3)
- new net R_BAT+: J?.1 (Pin_1), U?.15 (BAT+)
- new net R_BAT-: J?.2 (Pin_2), U?.16 (BAT-)
- new net R_C0: S?.1 (A), S?.1 (A), S?.1 (A), U?.1 (PA02_A0_D0)
- new net R_C1: S?.1 (A), S?.1 (A), S?.1 (A), U?.2 (PA4_A1_D1)
- new net R_C2: S?.1 (A), S?.1 (A), S?.1 (A), S?.1 (A), SW?.S2, U?.3 (PA10_A2_D2)
- new net R_C3: S?.1 (A), S?.1 (A), S?.1 (A), S?.1 (A), U?.4 (PA11_A3_D3)
- new net R_C4: S?.1 (A), S?.1 (A), S?.1 (A), S?.1 (A), U?.5 (PA8_A4_D4_SDA)
- new net R_GND: U?.13 (GND)
- new net R_R0: D?.1 (K), D?.1 (K), D?.1 (K), D?.1 (K), D?.1 (K), U?.11 (PA6_A10_D10_MOSI)
- new net R_R1: D?.1 (K), D?.1 (K), D?.1 (K), D?.1 (K), D?.1 (K), U?.10 (PA5_A9_D9_MISO)
- new net R_R2: D?.1 (K), D?.1 (K), D?.1 (K), D?.1 (K), D?.1 (K), U?.9 (PA7_A8_D8_SCK)
- new net R_R3: D?.1 (K), D?.1 (K), D?.1 (K), U?.8 (PB09_A7_D7_RX)
- new net R_RE-A: U?.7 (PB08_A6_D6_TX)
- new net R_RE-B: U?.6 (PA9_A5_D5_SCL)
- new net R_RE-C: JP?.2 (C)
- no-connect marks 4 -> 10
Other:
- moved on the sheet: D16, D17, D18, J1, JP1, S16, S17, S18, SW1, U1

Commit message: add stuff
Parts:
- JP1: value (none) -> RE_SJ
- gave numbers to parts that had none: 40
Connections:
- net L_GND: now also JP1.1 (A), U1.20 (GND)
- net L_RE-A: no longer SW2.A
- net L_RE-B: no longer SW2.B
- net L_RE-C: no longer SW2.C
- net R_GND: now also JP2.1 (A), U2.20 (GND)
- net R_RE-A: now also SW2.A
- net R_RE-B: now also SW2.B
- net R_RE-C: now also SW2.C
- removed net GND: JP1.1 (A), JP2.1 (A)
- no-connect marks 10 -> 8

Commit message: add stuff :/
Parts:
- removed D1, D10, D11, D12, D13, D14, D15, D16, D17, D18, D19, D2, D20, D21, D22, D23, D24, D25, D26, D27, D28, D29, D3, D30, D31, D32, D33, D34, D35, D36, D4, D5, D6, D7, D8, D9: 1N4148W, Diode_SMD:D_0805_2012Metric, symbol Device:D_Small_Filled
- removed JP1, JP2: RE_SJ, Jumper:SolderJumper-3_P2.0mm_Open_TrianglePad1.0x1.5mm, symbol Jumper:SolderJumper_3_Open
- removed S16, S34: SW_SPST, switches:Choc_PG1350_Choc_Spacing, symbol Switch:SW_SPST
- S1, S10, S11, S12, S13, S14, S15, S17, S18, S19, S2, S20, S21, S22, S23, S24, S25, S26, S27, S28, S29, S3, S30, S31, S32, S33, S35, S36, S4, S5, S6, S7, S8, S9: footprint switches:Choc_PG1350_Choc_Spacing -> reee:Choc_PG1350_Tight
- S16: renamed from SW1; footprint Encoder:RollerEncoder_Panasonic_EVQWGD001 -> reee:Choc_PG1350_Tight__EVQWGD001__Combo
- S34: renamed from SW2; footprint Encoder:RollerEncoder_Panasonic_EVQWGD001 -> reee:Choc_PG1350_Tight__EVQWGD001__Combo
Connections:
- net L_BAT- is gone; now on net L_GND: J1.2 (Pin_2), U1.16 (BAT-)
- net L_RE-C is gone; now on net L_GND: S16.C
- net R_BAT- is gone; now on net R_GND: J2.2 (Pin_2), U2.16 (BAT-)
- net R_RE-C is gone; now on net R_GND: S34.C
- net L_C2: now also S16.S1; no longer S16.S2
- net L_R0: now also S1.2 (B), S10.2 (B), S13.2 (B), S4.2 (B), S7.2 (B), U1.10 (PA5_A9_D9_MISO); no longer U1.11 (PA6_A10_D10_MOSI)
- net L_R1: now also S11.2 (B), S14.2 (B), S2.2 (B), S5.2 (B), S8.2 (B), U1.9 (PA7_A8_D8_SCK); no longer U1.10 (PA5_A9_D9_MISO)
- net L_R2: now also S12.2 (B), S15.2 (B), S3.2 (B), S6.2 (B), S9.2 (B), U1.8 (PB09_A7_D7_RX); no longer U1.9 (PA7_A8_D8_SCK)
- net L_R3: now also S16.S2, S17.2 (B), S18.2 (B), U1.11 (PA6_A10_D10_MOSI); no longer U1.8 (PB09_A7_D7_RX)
- net R_C2: now also S34.S1; no longer S34.S2
- net R_R0: now also S19.2 (B), S22.2 (B), S25.2 (B), S28.2 (B), S31.2 (B), U2.10 (PA5_A9_D9_MISO); no longer U2.11 (PA6_A10_D10_MOSI)
- net R_R1: now also S20.2 (B), S23.2 (B), S26.2 (B), S29.2 (B), S32.2 (B), U2.9 (PA7_A8_D8_SCK); no longer U2.10 (PA5_A9_D9_MISO)
- net R_R2: now also S21.2 (B), S24.2 (B), S27.2 (B), S30.2 (B), S33.2 (B), U2.8 (PB09_A7_D7_RX); no longer U2.9 (PA7_A8_D8_SCK)
- net R_R3: now also S34.S2, S35.2 (B), S36.2 (B), U2.11 (PA6_A10_D10_MOSI); no longer U2.8 (PB09_A7_D7_RX)
Other:
- moved on the sheet: S16, S34
